File: base/mosfets_sens_isol.sch (KiCad schematic (older format))
At the start: 81 parts, among them Q1 irf540n, Q2 irf540n, Q3 irf540n, Q4 irf540n, Q5 irf540n, Q6 irf540n, Q7 irf540n, Q8 irf540n, U1 SI8640, U10 ADS7886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

Commit message: current pcb
Parts:
- removed D1, D2, D3, D4: bav21, Package_TO_SOT_SMD:SOT-23, symbol D
- added D1, D2, D3, D4: D_Schottky_AKK, Package_TO_SOT_SMD:SOT-23, symbol D_Schottky_AKK
Other:
- moved on the sheet: C5, C6, C7, C8, TP27, TP28
Changed lines of the file:
@@
 L C_Small C5
 U 1 1 5A1E0E58
-P 5400 1300
-F 0 "C5" V 5500 1250 50  0000 L CNN
-F 1 "1uF 50V" V 5300 1200 39  0000 L CNN
-F 2 "Capacitor_SMD:C_0805_2012Metric" H 5400 1300 50  0001 C CNN
-F 3 "" H 5400 1300 50  0001 C CNN
-	1    5400 1300
+P 5500 1300
+F 0 "C5" V 5600 1250 50  0000 L CNN
+F 1 "1uF 50V" V 5400 1200 39  0000 L CNN
+F 2 "Capacitor_SMD:C_0805_2012Metric" H 5500 1300 50  0001 C CNN
+F 3 "" H 5500 1300 50  0001 C CNN
+	1    5500 1300
 	0    -1   -1   0
-$EndComp
-$Comp
-L D D1
-U 1 1 5A1E0FA3
-P 5000 1300
-F 0 "D1" H 5000 1200 50  0000 C CNN
-F 1 "bav21" H 5000 1400 50  0001 C CNN
-F 2 "Package_TO_SOT_SMD:SOT-23" H 5000 1300 50  0001 C CNN
-F 3 "" H 5000 1300 50  0001 C CNN
-	1    5000 1300
-	-1   0    0    1
 $EndComp
 Text Label 1300 900  0    60   ~ 0
@@
 $EndComp
 $Comp
-L IR2181 U4
-U 1 1 5A25F1D0
-P 4800 3300
-F 0 "U4" H 4850 3750 50  0000 L CNN
-F 1 "IR2181" H 4850 2850 50  0000 L CNN
-F 2 "Package_SOIC:SOIC-8_3.9x4.9mm_P1.27mm" H 4800 3300 50  0001 C CIN
-F 3 "" H 4800 3300 50  0001 C CNN
-	1    4800 3300
-	1    0    0    -1
-$EndComp
-$Comp
 L R R11
 U 1 1 5A25F1D6
@@
 L C_Small C6
 U 1 1 5A25F1E2
-P 5450 2750
-F 0 "C6" V 5550 2700 50  0000 L CNN
-F 1 "1uF 50V" V 5350 2550 50  0000 L CNN
-F 2 "Capacitor_SMD:C_0805_2012Metric" H 5450 2750 50  0001 C CNN
-F 3 "" H 5450 2750 50  0001 C CNN
-	1    5450 2750
+P 5550 2750
+F 0 "C6" V 5650 2700 50  0000 L CNN
+F 1 "1uF 50V" V 5450 2550 50  0000 L CNN
+F 2 "Capacitor_SMD:C_0805_2012Metric" H 5550 2750 50  0001 C CNN
+F 3 "" H 5550 2750 50  0001 C CNN
+	1    5550 2750
 	0    -1   -1   0
-$EndComp
-$Comp
-L D D2
-U 1 1 5A25F1E8
-P 5100 2750
-F 0 "D2" H 5100 2650 50  0000 C CNN
-F 1 "bav21" H 5100 2850 50  0001 C CNN
-F 2 "Package_TO_SOT_SMD:SOT-23" H 5100 2750 50  0001 C CNN
-F 3 "" H 5100 2750 50  0001 C CNN
-	1    5100 2750
-	-1   0    0    1
 $EndComp
 $Comp
@@
 L C_Small C7
 U 1 1 5A25F66C
-P 5450 4200
-F 0 "C7" V 5550 4150 50  0000 L CNN
-F 1 "1uF 50V" V 5350 4000 50  0000 L CNN
-F 2 "Capacitor_SMD:C_0805_2012Metric" H 5450 4200 50  0001 C CNN
-F 3 "" H 5450 4200 50  0001 C CNN
-	1    5450 4200
+P 5550 4200
+F 0 "C7" V 5650 4150 50  0000 L CNN
+F 1 "1uF 50V" V 5450 4000 50  0000 L CNN
+F 2 "Capacitor_SMD:C_0805_2012Metric" H 5550 4200 50  0001 C CNN
+F 3 "" H 5550 4200 50  0001 C CNN
+	1    5550 4200
 	0    -1   -1   0
-$EndComp
-$Comp
-L D D3
-U 1 1 5A25F672
-P 5100 4200
-F 0 "D3" H 5100 4100 50  0000 C CNN
-F 1 "bav21" H 5100 4300 50  0001 C CNN
-F 2 "Package_TO_SOT_SMD:SOT-23" H 5100 4200 50  0001 C CNN
-F 3 "" H 5100 4200 50  0001 C CNN
-	1    5100 4200
-	-1   0    0    1
 $EndComp
 $Comp
@@
 L C_Small C8
 U 1 1 5A25F6C6
-P 5450 5650
-F 0 "C8" V 5550 5600 50  0000 L CNN
-F 1 "1uF 50V" V 5350 5450 50  0000 L CNN
-F 2 "Capacitor_SMD:C_0805_2012Metric" H 5450 5650 50  0001 C CNN
-F 3 "" H 5450 5650 50  0001 C CNN
-	1    5450 5650
+P 5550 5650
+F 0 "C8" V 5650 5600 50  0000 L CNN
+F 1 "1uF 50V" V 5450 5450 50  0000 L CNN
+F 2 "Capacitor_SMD:C_0805_2012Metric" H 5550 5650 50  0001 C CNN
+F 3 "" H 5550 5650 50  0001 C CNN
+	1    5550 5650
 	0    -1   -1   0
-$EndComp
-$Comp
-L D D4
-U 1 1 5A25F6CC
-P 5100 5650
-F 0 "D4" H 5100 5550 50  0000 C CNN
-F 1 "bav21" H 5100 5750 50  0001 C CNN
-F 2 "Package_TO_SOT_SMD:SOT-23" H 5100 5650 50  0001 C CNN
-F 3 "" H 5100 5650 50  0001 C CNN
-	1    5100 5650
-	-1   0    0    1
 $EndComp
 $Comp
@@
 L Test_Point TP28
 U 1 1 5A4A934F
-P 5600 1000
-F 0 "TP28" H 5600 1270 50  0000 C CNN
-F 1 "driver_VS" H 5600 1200 50  0000 C CNN
-F 2 "TestPoint:TestPoint_Pad_D1.5mm" H 5800 1000 50  0001 C CNN
-F 3 "" H 5800 1000 50  0001 C CNN
-	1    5600 1000
+P 5650 1000
+F 0 "TP28" H 5650 1300 50  0000 C CNN
+F 1 "driver_VS" H 5650 1200 50  0000 C CNN
+F 2 "TestPoint:TestPoint_Pad_D1.5mm" H 5850 1000 50  0001 C CNN
+F 3 "" H 5850 1000 50  0001 C CNN
+	1    5650 1000
 	1    0    0    -1
 $EndComp
@@
 L Test_Point TP27
 U 1 1 5A4A9424
-P 5200 1000
-F 0 "TP27" H 5200 1270 50  0000 C CNN
-F 1 "driver_VB" H 5200 1200 50  0000 C CNN
-F 2 "TestPoint:TestPoint_Pad_D1.5mm" H 5400 1000 50  0001 C CNN
-F 3 "" H 5400 1000 50  0001 C CNN
-	1    5200 1000
+P 5350 1000
+F 0 "TP27" H 5250 1300 50  0000 C CNN
+F 1 "driver_VB" H 5150 1200 50  0000 C CNN
+F 2 "TestPoint:TestPoint_Pad_D1.5mm" H 5550 1000 50  0001 C CNN
+F 3 "" H 5550 1000 50  0001 C CNN
+	1    5350 1000
 	1    0    0    -1
 $EndComp
@@
 U 1 1 5A4AA2DB
 P 6000 1000
-F 0 "TP29" H 6000 1270 50  0000 C CNN
-F 1 "driver_HO" H 6000 1200 50  0000 C CNN
+F 0 "TP29" H 6000 1300 50  0000 C CNN
+F 1 "driver_HO" H 6050 1200 50  0000 C CNN
 F 2 "TestPoint:TestPoint_Pad_D1.5mm" H 6200 1000 50  0001 C CNN
 F 3 "" H 6200 1000 50  0001 C CNN
@@
 	5700 5650 5700 6250
 Wire Wire Line
-	5550 5650 5700 5650
-Connection ~ 5300 5650
+	5650 5650 5700 5650
+Connection ~ 5400 5650
 Wire Wire Line
 	6600 6750 6600 6650
@@
 	4800 5650 4800 5700
 Wire Wire Line
-	4250 5650 4950 5650
-Wire Wire Line
-	5300 5650 5300 5900
-Wire Wire Line
-	5250 5650 5350 5650
+	4250 5650 4900 5650
+Wire Wire Line
+	5400 5650 5400 5900
+Wire Wire Line
+	5350 5650 5450 5650
 Connection ~ 6050 5650
 Wire Wire Line
@@
 Connection ~ 4800 6750
 Wire Wire Line
-	5300 5900 5100 5900
+	5400 5900 5100 5900
 Wire Wire Line
 	5150 6400 5150 6250
@@
 	5700 4200 5700 4800
 Wire Wire Line
-	5550 4200 5700 4200
-Connection ~ 5300 4200
+	5650 4200 5700 4200
+Connection ~ 5400 4200
 Wire Wire Line
 	6600 5300 6600 5200
@@
 	4800 4200 4800 4250
 Wire Wire Line
-	4250 4200 4950 4200
-Wire Wire Line
-	5300 4200 5300 4450
-Wire Wire Line
-	5250 4200 5350 4200
+	5400 4200 5400 4450
 Connection ~ 6050 4200
 Wire Wire Line
@@
 Connection ~ 4800 5300
 Wire Wire Line
-	5300 4450 5100 4450
+	5400 4450 5100 4450
 Wire Wire Line
 	5150 4950 5150 4800
@@
 	5700 2750 5700 3350
 Wire Wire Line
-	5550 2750 5700 2750
-Connection ~ 5300 2750
+	5650 2750 5700 2750
+Connection ~ 5400 2750
 Wire Wire Line
 	6600 3850 6600 3750
@@
 	6600 2750 6600 2950
 Connection ~ 6050 3850
-Connection ~ 4800 2750
-Wire Wire Line
-	4800 2750 4800 2800
-Wire Wire Line
-	4250 2750 4950 2750
-Wire Wire Line
-	5300 2750 5300 3000
-Wire Wire Line
-	5250 2750 5350 2750
+Wire Wire Line
+	5400 2750 5400 3000
+Wire Wire Line
+	5350 2750 5450 2750
 Connection ~ 6050 2750
 Wire Wire Line
@@
 Connection ~ 4800 3850
 Wire Wire Line
-	5300 3000 5100 3000
+	5400 3000 5100 3000
 Wire Wire Line
 	5150 3500 5150 3350
@@
 Wire Wire Line
 	6050 1300 6850 1300
-Connection ~ 5600 1900
-Wire Wire Line
-	5600 1000 5600 1900
-Wire Wire Line
-	5500 1300 5600 1300
-Connection ~ 5200 1300
+Connection ~ 5650 1900
+Wire Wire Line
+	5650 1000 5650 1900
+Wire Wire Line
+	5600 1300 5650 1300
+Connection ~ 5350 1300
 Connection ~ 10100 5800
 Connection ~ 10100 5350
@@
 	4250 1300 4850 1300
 Wire Wire Line
-	5200 1000 5200 1550
-Wire Wire Line
-	5150 1300 5300 1300
+	5350 1000 5350 1550
 Wire Wire Line
 	6050 1450 6050 1300
@@
 	1100 900  1550 900
 Wire Wire Line
-	5200 1550 5100 1550
+	5350 1550 5100 1550
 Wire Wire Line
 	5150 2050 5150 1900
@@
 Wire Notes Line
 	8250 2950 8250 2650
-Connection ~ 5600 1300
+Connection ~ 5650 1300
 Connection ~ 5750 1650
 Connection ~ 6600 1300
@@
 Wire Wire Line
 	6000 1050 6000 1000
+$Comp
+L D_Schottky_AKK D1
+U 1 1 5A690E26
+P 5050 1300
+F 0 "D1" H 5050 1400 50  0000 C CNN
+F 1 "D_Schottky_AKK" H 5050 1200 50  0000 C CNN
+F 2 "Package_TO_SOT_SMD:SOT-23" H 5050 1300 50  0001 C CNN
+F 3 "" H 5050 1300 50  0001 C CNN
+	1    5050 1300
+	-1   0    0    1
+$EndComp
+Wire Wire Line
+	5300 1300 5400 1300
+$Comp
+L D_Schottky_AKK D2
+U 1 1 5A6A5C15
+P 5100 2750
+F 0 "D2" H 5100 2850 50  0000 C CNN
+F 1 "D_Schottky_AKK" H 5100 2650 50  0000 C CNN
+F 2 "Package_TO_SOT_SMD:SOT-23" H 5100 2750 50  0001 C CNN
+F 3 "" H 5100 2750 50  0001 C CNN
+	1    5100 2750
+	-1   0    0    1
+$EndComp
+Wire Wire Line
+	5350 4200 5450 4200
+$Comp
+L IR2181 U4
+U 1 1 5A25F1D0
+P 4800 3300
+F 0 "U4" H 4850 3750 50  0000 L CNN
+F 1 "IR2181" H 4850 2850 50  0000 L CNN
+F 2 "Package_SOIC:SOIC-8_3.9x4.9mm_P1.27mm" H 4800 3300 50  0001 C CIN
+F 3 "" H 4800 3300 50  0001 C CNN
+	1    4800 3300
+	1    0    0    -1
+$EndComp
+Wire Wire Line
+	4250 2750 4900 2750
+Wire Wire Line
+	4800 2800 4800 2750
+Connection ~ 4800 2750
+$Comp
+L D_Schottky_AKK D3
+U 1 1 5A6A87E9
+P 5100 4200
+F 0 "D3" H 5100 4300 50  0000 C CNN
+F 1 "D_Schottky_AKK" H 5100 4100 50  0000 C CNN
+F 2 "Package_TO_SOT_SMD:SOT-23" H 5100 4200 50  0001 C CNN
+F 3 "" H 5100 4200 50  0001 C CNN
+	1    5100 4200
+	-1   0    0    1
+$EndComp
+Wire Wire Line
+	4250 4200 4900 4200
+$Comp
+L D_Schottky_AKK D4
+U 1 1 5A6A94B7
+P 5100 5650
+F 0 "D4" H 5100 5750 50  0000 C CNN
+F 1 "D_Schottky_AKK" H 5100 5550 50  0000 C CNN
+F 2 "Package_TO_SOT_SMD:SOT-23" H 5100 5650 50  0001 C CNN
+F 3 "" H 5100 5650 50  0001 C CNN
+	1    5100 5650
+	-1   0    0    1
+$EndComp
 $EndSCHEMATC
