File: base/can_rs485.sch (KiCad schematic (older format))
At the start: 15 parts, among them U20 SN65HVD230, U21 MAX485CSA

Commit message: upd
Parts:
- renumbered C42 to C40, C43 to C41
Changed lines of the file:
@@
 	3500 2400 5000 2400
 $Comp
-L C C42
+L C C40
 U 1 1 5A3C342C
 P 1500 1150
-F 0 "C42" H 1525 1250 50  0000 L CNN
+F 0 "C40" H 1525 1250 50  0000 L CNN
 F 1 "0.1uF" H 1525 1050 50  0000 L CNN
 F 2 "Capacitor_SMD:C_0603_1608Metric" H 1538 1000 50  0001 C CNN
@@
 	5000 6000 5000 6150
 $Comp
-L C C43
+L C C41
 U 1 1 5A44D127
 P 2200 4850
-F 0 "C43" H 2225 4950 50  0000 L CNN
+F 0 "C41" H 2225 4950 50  0000 L CNN
 F 1 "0.1uF" H 2225 4750 50  0000 L CNN
 F 2 "Capacitor_SMD:C_0603_1608Metric" H 2238 4700 50  0001 C CNN
