File: base/mcu_fpga_con.sch (KiCad schematic (older format))
At the start: 2 parts, among them J14 Conn_02x25_Odd_Even, J15 Conn_02x25_Odd_Even

Commit message: upd
Parts:
- renumbered J14 to J15, J15 to J16
Changed lines of the file:
@@
 Vsense1
 $Comp
-L Conn_02x25_Odd_Even J14
+L Conn_02x25_Odd_Even J15
 U 1 1 5A2BAF82
 P 4000 2600
-F 0 "J14" H 4050 3900 50  0000 C CNN
+F 0 "J15" H 4050 3900 50  0000 C CNN
 F 1 "Conn_02x25_Odd_Even" H 4050 1300 50  0000 C CNN
 F 2 "Connector_PinHeader_2.54mm:PinHeader_2x25_P2.54mm_Vertical" H 4000 2600 50  0001 C CNN
@@
 $EndComp
 $Comp
-L Conn_02x25_Odd_Even J15
+L Conn_02x25_Odd_Even J16
 U 1 1 5A2BB01B
 P 6700 2600
-F 0 "J15" H 6750 3900 50  0000 C CNN
+F 0 "J16" H 6750 3900 50  0000 C CNN
 F 1 "Conn_02x25_Odd_Even" H 6750 1300 50  0000 C CNN
 F 2 "Connector_PinHeader_2.54mm:PinHeader_2x25_P2.54mm_Vertical" H 6700 2600 50  0001 C CNN

Commit message: upd
Parts:
- removed J15, J16: Conn_02x25_Odd_Even, Connector_PinHeader_2.54mm:PinHeader_2x25_P2.54mm_Vertical, symbol Conn_02x25_Odd_Even
- added J15, J16: Conn_01x27, Connector_PinHeader_2.54mm:PinHeader_1x27_P2.54mm_Vertical, symbol Conn_01x27
Connections:
- net labels removed: CAN_RX, CAN_TX, RS485_RX, RS485_TX, RS485_TXEX, SPI0_CSn, SPI0_MISO, SPI0_SCK, SPI1_CSn, SPI1_MISO, SPI1_SCK
- wire segments 53 -> 58
