File: base/4hbd-base.kicad_pcb (KiCad board)
At the start: 2 copper layers, 182 x 100 mm, 233 parts, among them J1 Spring_Terminal_Connector_01x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, J10 Spring_Terminal_Connector_01x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, J11 Spring_Terminal_Connector_01x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, J12 Spring_Terminal_Connector_01x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, J13 Screw_Terminal_01x02, J14 Conn_02x25_Odd_Even, J15 Conn_02x25_Odd_Even, J2 Spring_Terminal_Connector_01x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, J3 Spring_Terminal_Connector_01x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, J4 Spring_Terminal_Connector_01x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, J5 Spring_Terminal_Connector_01x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, J6 Spring_Terminal_Connector_01x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, J7 Screw_Terminal_01x03, J8 Screw_Terminal_01x04, J9 Spring_Terminal_Connector_01x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, Q1 irf540n, Q10 2N7002, Q11 2N7002, Q12 IRLML2060TRPBF, Q2 irf540n, Q3 irf540n, Q4 irf540n, Q5 irf540n, Q6 irf540n, Q7 irf540n, Q8 irf540n, Q9 2N7002, U1 SI8640, U10 ADS7886, U11 MOCD217M, U12 MOCD217M, U13 MOCD217M, U14 AMS1117-5.0, U15 AMS1117-5.0, U16 LM2596S-ADJ, U17 AM26LV32, U18 LM2596S-ADJ, U19 AMS1117-5.0, U2 SI8640, U20 SN65HVD230, U21 MAX485CSA, U3 IR2181, U4 IR2181, U5 IR2181, U6 IR2181, U7 ACS712xLCTR-30A, U8 ACS712xLCTR-30A, U9 ADS7886

Commit message: current pcb
Parts:
- D1, D2, D3, D4: value bav21 -> D_Schottky_AKK
- J1, J10, J11, J12, J13, J14, J15, J2, J3, J4, J5, J6, J7, J8, J9, Q1, Q2, Q3, Q4, Q5, Q6, Q7, Q8, R35, R36: moved to B.Cu
- MK1, MK2, MK3, MK4: footprint MountingHole:MountingHole_3.5mm_Pad -> MountingHole:MountingHole_3.5mm
- moved U19 332.2 mm to (24.5, 113.9), turned to 180 degrees
- moved C41 319.9 mm to (47.1, 120.2)
- moved D29 316.0 mm to (66.8, 133.7), turned to 180 degrees
- moved R51 315.6 mm to (74.8, 122.4), turned to 90 degrees
- moved R52 313.0 mm to (74.9, 125.1), turned to 180 degrees
- moved R50 312.5 mm to (77.6, 124.3), turned to 270 degrees
- moved D28 306.8 mm to (68.7, 139.9), turned to 270 degrees
- moved C17 296.3 mm to (61.8, 114.6)
- moved C37 295.4 mm to (72.0, 133.0), turned to 270 degrees
- moved D30 295.2 mm to (87.0, 131.0)
- moved C7 284.6 mm to (80.0, 111.8), turned to 180 degrees
- moved R14 284.0 mm to (72.8, 101.1), turned to 270 degrees
- moved R15 281.6 mm to (68.8, 105.1), turned to 270 degrees
- moved R16 273.2 mm to (58.8, 101.1), turned to 270 degrees
- moved R12 273.0 mm to (86.8, 101.1), turned to 270 degrees
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Connections:
- D1 pad 1: Net-(C5-Pad1) -> /DIO/+12V
- D1 pad 2: /DIO/+12V -> (no net)
- D1 pad 3: (no net) -> Net-(C5-Pad1)
- D2 pad 1: Net-(C6-Pad1) -> /DIO/+12V
- D2 pad 2: /DIO/+12V -> (no net)
- D2 pad 3: (no net) -> Net-(C6-Pad1)
- D3 pad 1: Net-(C7-Pad1) -> /DIO/+12V
- D3 pad 2: /DIO/+12V -> (no net)
- D3 pad 3: (no net) -> Net-(C7-Pad1)
- D4 pad 1: Net-(C8-Pad1) -> /DIO/+12V
- D4 pad 2: /DIO/+12V -> (no net)
- D4 pad 3: (no net) -> Net-(C8-Pad1)
- J13 pad 1: /Digital DC/DC/+24VD -> GND
- J13 pad 2: GND -> /Digital DC/DC/+24VD
- J7 pad 1: /MOSFETs/CurSense/Isolation/Vpwr -> GNDPWR
- J7 pad 2: /Power DC/DC/+24VP -> /MOSFETs/CurSense/Isolation/Vpwr
- J7 pad 3: GNDPWR -> /Power DC/DC/+24VP
- U10 pad 1: Net-(R18-Pad2) -> /CAN/RS485/+5V
- U10 pad 3: (no net) -> Net-(R18-Pad2)
- U9 pad 1: Net-(R17-Pad2) -> /CAN/RS485/+5V
- U9 pad 3: (no net) -> Net-(R17-Pad2)
Routing:
- net GNDPWR: track 0.00 -> 107.5 mm
- net /MOSFETs/CurSense/Isolation/Vpwr: track 0.00 -> 102.4 mm
- net /DIO/+12V: track 0.00 -> 80.2 mm
- net /MOSFETs/CurSense/Isolation/HB0: track 0.00 -> 32.0 mm
- net /MOSFETs/CurSense/Isolation/HB2: track 0.00 -> 29.0 mm
- net /MOSFETs/CurSense/Isolation/HB3: track 0.00 -> 28.9 mm
- net /MOSFETs/CurSense/Isolation/HB1: track 0.00 -> 24.6 mm
- net Net-(C24-Pad1): track 0.00 -> 17.1 mm
- net Net-(C30-Pad1): track 0.00 -> 13.1 mm
- net Net-(R10-Pad2): track 0.00 -> 12.2 mm
- net Net-(R14-Pad2): track 0.00 -> 12.0 mm
- net Net-(R12-Pad2): track 0.00 -> 12.0 mm
- net Net-(R16-Pad2): track 0.00 -> 12.0 mm
- net Net-(C8-Pad1): track 0.00 -> 10.1 mm
- net Net-(C7-Pad1): track 0.00 -> 10.1 mm
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- added copper zone on F.Cu, net /MOSFETs/CurSense/Isolation/HB0
- added copper zone on F.Cu, net /MOSFETs/CurSense/Isolation/HB0s
- added copper zone on F.Cu, net /MOSFETs/CurSense/Isolation/HB1
- added copper zone on F.Cu, net /MOSFETs/CurSense/Isolation/HB2
- added copper zone on F.Cu, net /MOSFETs/CurSense/Isolation/HB2s
- added copper zone on F.Cu, net /MOSFETs/CurSense/Isolation/HB3
Other:
- net class Default: clearance 0.2 -> 0.4; trace_width 0.25 -> 0.4; via_dia 0.6 -> 0.8
- rule trace_clearance: 0.2 -> 0.4
- rule trace_min: 0.2 -> 0.4
- rule via_min_drill: 0.3 -> 0.4
- rule via_min_size: 0.4 -> 0.7

Commit message: upd adc
Parts:
- removed C42, C43: 0.1uF, Capacitor_SMD:C_0603_1608Metric
- added J16: Conn_02x25_Odd_Even, Connector_PinHeader_2.54mm:PinHeader_2x25_P2.54mm_Vertical, F.Cu at (134.8, 74.0)
- C17, C18: footprint Capacitor_SMD:C_0603_1608Metric -> Capacitor_SMD:C_0805_2012Metric
- C20, C21: value 0.1uF -> 22uF 10V; footprint Capacitor_SMD:C_0805_2012Metric -> Capacitor_Tantalum_SMD:CP_EIA-3216-18_Kemet-A
- C22: value 22uF 10V -> 3.3nF 50V; footprint Capacitor_Tantalum_SMD:CP_EIA-3216-18_Kemet-A -> Capacitor_SMD:C_0603_1608Metric
- C23: value 22uF 10V -> 220uF 35V; footprint Capacitor_Tantalum_SMD:CP_EIA-3216-18_Kemet-A -> Capacitor_SMD:CP_Elec_8x10
- C24: value 3.3nF 50V -> 22uF 6.3V; footprint Capacitor_SMD:C_0603_1608Metric -> Capacitor_Tantalum_SMD:CP_EIA-3216-18_Kemet-A
- C25: value 220uF 35V -> 22uF 6.3V; footprint Capacitor_SMD:CP_Elec_8x10 -> Capacitor_Tantalum_SMD:CP_EIA-3216-18_Kemet-A
- C26, C27: value 22uF 6.3V -> 4.7uF 6.3V; footprint Capacitor_Tantalum_SMD:CP_EIA-3216-18_Kemet-A -> Capacitor_SMD:C_0603_1608Metric
- C28: value 4.7uF 6.3V -> 220uF 35V; footprint Capacitor_SMD:C_0603_1608Metric -> Capacitor_SMD:CP_Elec_8x10
- C29: value 4.7uF 6.3V -> 4.7uF 50V; footprint Capacitor_SMD:C_0603_1608Metric -> Capacitor_SMD:C_1210_3225Metric
- C30: value 220uF 35V -> 4.7uF 50V; footprint Capacitor_SMD:CP_Elec_8x10 -> Capacitor_SMD:C_1210_3225Metric
- C31, C32: value 4.7uF 50V -> 470uF 10V; footprint Capacitor_SMD:C_1210_3225Metric -> Capacitor_SMD:CP_Elec_8x10
- C33, C34: value 470uF 10V -> 0.1uF; footprint Capacitor_SMD:CP_Elec_8x10 -> Capacitor_SMD:C_0603_1608Metric
- C35: value 0.1uF -> 3.3nF 50V
- C36: value 0.1uF -> 100uF 35V; footprint Capacitor_SMD:C_0603_1608Metric -> Capacitor_SMD:CP_Elec_6.3x7.7
- C37: value 3.3nF 50V -> 100uF 16V; footprint Capacitor_SMD:C_0603_1608Metric -> Capacitor_SMD:CP_Elec_6.3x5.3
- C38: value 100uF 35V -> 220uF 10V; footprint Capacitor_SMD:CP_Elec_6.3x7.7 -> Capacitor_SMD:CP_Elec_6.3x5.3
- C39: value 100uF 16V -> 4.7uF 6.3V; footprint Capacitor_SMD:CP_Elec_6.3x5.3 -> Capacitor_SMD:C_0603_1608Metric
- C40: value 220uF 10V -> 0.1uF; footprint Capacitor_SMD:CP_Elec_6.3x5.3 -> Capacitor_SMD:C_0603_1608Metric
- C41: value 4.7uF 6.3V -> 0.1uF
- J12: value Spring_Terminal_Connector_01x08 -> Spring_Terminal_Connector_01x03; footprint TerminalBlock_KaiFeng:TerminalBlock_KaiFeng_KF141R-8_1x08_P2.54mm -> TerminalBlock_KaiFeng:TerminalBlock_KaiFeng_KF141R-3_1x03_P2.54mm
- J13: value Screw_Terminal_01x02 -> Spring_Terminal_Connector_01x08; footprint TerminalBlock:TerminalBlock_Altech_AK300-2_P5.00mm -> TerminalBlock_KaiFeng:TerminalBlock_KaiFeng_KF141R-8_1x08_P2.54mm
- J14: value Conn_02x25_Odd_Even -> Screw_Terminal_01x02; footprint Connector_PinHeader_2.54mm:PinHeader_2x25_P2.54mm_Vertical -> TerminalBlock:TerminalBlock_Altech_AK300-2_P5.00mm
- J7: value Screw_Terminal_01x03 -> Screw_Terminal_01x02; footprint TerminalBlock:TerminalBlock_Altech_AK300-3_P5.00mm -> TerminalBlock:TerminalBlock_Altech_AK300-2_P5.00mm
- J8: value Screw_Terminal_01x04 -> Screw_Terminal_01x02; footprint TerminalBlock:TerminalBlock_Altech_AK300-4_P5.00mm -> TerminalBlock:TerminalBlock_Altech_AK300-2_P5.00mm
- J9: value Spring_Terminal_Connector_01x03 -> Screw_Terminal_01x04; footprint TerminalBlock_KaiFeng:TerminalBlock_KaiFeng_KF141R-3_1x03_P2.54mm -> TerminalBlock:TerminalBlock_Altech_AK300-4_P5.00mm
- U3, U4, U5, U6: value IR2181 -> IR25606
- moved TP27 308.7 mm to (-193.0, 165.5), turned to 90 degrees
- moved R45 205.5 mm to (121.1, 220.7)
- moved R46 205.5 mm to (124.6, 220.4)
- moved U14 168.1 mm to (155.6, 130.2), turned to 180 degrees
- moved C28 153.9 mm to (161.8, 133.2), turned to 270 degrees
- moved C22 150.8 mm to (163.2, 127.8)
- moved C26 142.8 mm to (163.2, 130.2)
- moved J13 117.6 mm to (153.0, 24.2), turned to 180 degrees
- moved C35 111.2 mm to (159.7, 121.9)
- moved D26 110.2 mm to (164.9, 106.3)
- moved D27 107.2 mm to (160.5, 118.9)
- moved L4 106.9 mm to (160.3, 124.9)
- moved C34 105.4 mm to (152.1, 121.9), turned to 180 degrees
- moved J9 102.2 mm to (57.6, 105.2), turned to 90 degrees
- moved J11 100.9 mm to (67.0, 25.0)
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Connections:
- C13 pad 1: Net-(C13-Pad1) -> GNDPWR
- C13 pad 2: GND -> /DIO/+12V
- C14 pad 1: Net-(C14-Pad1) -> GND
- C14 pad 2: GND -> /CAN/RS485/+5V
- C17 pad 1: GNDPWR -> /TempSens/Fan/TempAnalog
- C17 pad 2: /DIO/+12V -> GND
- C18 pad 1: GND -> /TempSens/Fan/TempAnalog_2
- C18 pad 2: /CAN/RS485/+5V -> GND
- C19 pad 1: /TempSens/Fan/TempAnalog -> /MCU/FPGA connection/Vsense2
- C20 pad 1: /TempSens/Fan/TempAnalog_2 -> /Digital DC/DC/+6.8V
- C21 pad 1: /MCU/FPGA connection/Vsense2 -> /Digital DC/DC/+6.8V
- C22 pad 1: /Digital DC/DC/+6.8V -> Net-(C22-Pad1)
- C23 pad 1: /Digital DC/DC/+6.8V -> Net-(C22-Pad1)
- C24 pad 1: Net-(C24-Pad1) -> /CAN/RS485/+5V
- C25 pad 1: Net-(C24-Pad1) -> /Digital DC/DC/+5VEnc
- C28 pad 1: /CAN/RS485/+5V -> Net-(C28-Pad1)
- C29 pad 1: /Digital DC/DC/+5VEnc -> Net-(C28-Pad1)
- C30 pad 1: Net-(C30-Pad1) -> /Digital DC/DC/+Vpp
- C31 pad 1: Net-(C30-Pad1) -> Net-(C31-Pad1)
- C32 pad 1: /Digital DC/DC/+Vpp -> Net-(C31-Pad1)
- C33 pad 1: Net-(C33-Pad1) -> Net-(C31-Pad1)
- C34 pad 1: Net-(C33-Pad1) -> +3V3
- C35 pad 1: Net-(C33-Pad1) -> Net-(C35-Pad1)
- C35 pad 2: GND -> GNDPWR
- C36 pad 1: +3V3 -> Net-(C35-Pad1)
- C36 pad 2: GND -> GNDPWR
- C37 pad 1: Net-(C37-Pad1) -> /DIO/+12V
- C38 pad 1: Net-(C37-Pad1) -> /MOSFETs/CurSense/Isolation/+5Vpwr
- C39 pad 1: /DIO/+12V -> /MOSFETs/CurSense/Isolation/+5Vpwr
- C40 pad 1: /MOSFETs/CurSense/Isolation/+5Vpwr -> +3V3
- C40 pad 2: GNDPWR -> GND
- C41 pad 1: /MOSFETs/CurSense/Isolation/+5Vpwr -> /CAN/RS485/+5V
- C41 pad 2: GNDPWR -> GND
- D24 pad 1: Net-(C24-Pad1) -> Net-(C22-Pad1)
- D25 pad 1: Net-(C30-Pad1) -> Net-(C28-Pad1)
- D27 pad 1: Net-(C33-Pad1) -> Net-(C31-Pad1)
- D28 pad 1: Net-(C37-Pad1) -> Net-(C35-Pad1)
- D29 pad 1: Net-(C37-Pad1) -> Net-(C35-Pad1)
- F3 pad 1: Net-(C24-Pad1) -> Net-(C22-Pad1)
- J10 pad 1: /CAN/RS485/RS485+ -> /CAN/RS485/CAN_H
- J10 pad 2: /CAN/RS485/RS485- -> /CAN/RS485/CAN_L
- J11 pad 1: /TempSens/Fan/FAN_PWR -> /CAN/RS485/RS485+
- J11 pad 2: GND -> /CAN/RS485/RS485-
- J11 pad 3: /TempSens/Fan/FAN_PULSE -> GND
- J12 pad 1: /Digital DC/DC/+5VEnc -> /TempSens/Fan/FAN_PWR
- J12 pad 3: /Encoder Interface/EncA+ -> /TempSens/Fan/FAN_PULSE
- J13 pad 1: GND -> /Digital DC/DC/+5VEnc
- J13 pad 2: /Digital DC/DC/+24VD -> GND
- J14 pad 1: (no net) -> GND
- J14 pad 2: (no net) -> /Digital DC/DC/+24VD
- J15 pad 1: /MCU/FPGA connection/SPI1_CSn -> (no net)
- J15 pad 10: (no net) -> GND
- J15 pad 11: (no net) -> +3V3
- J15 pad 13: /MCU/FPGA connection/PWM -> (no net)
- J15 pad 15: (no net) -> /MCU/FPGA connection/ADC_Csens0
- J15 pad 17: (no net) -> /MCU/FPGA connection/ADC_Csens1
- J15 pad 19: (no net) -> +3V3
- J15 pad 2: /MCU/FPGA connection/SPI1_SCK -> (no net)
- J15 pad 22: (no net) -> +3V3
- J15 pad 23: +3V3 -> /Encoder Interface/EncA
- J15 pad 24: GND -> /Encoder Interface/EncB
- J15 pad 25: +3V3 -> /Encoder Interface/EncZ
- J15 pad 27: (no net) -> GND
- J15 pad 28: (no net) -> +3V3
- J15 pad 29: (no net) -> /MCU/FPGA connection/SPI0_CSn
- J15 pad 3: /MCU/FPGA connection/SPI1_MISO -> (no net)
- J15 pad 30: (no net) -> /MCU/FPGA connection/SPI0_SCK
- J15 pad 31: /DIO/DI0 -> /MCU/FPGA connection/SPI0_MISO
- J15 pad 32: /DIO/DI1 -> (no net)
- J15 pad 33: /DIO/DI2 -> /MCU/FPGA connection/Vsense2
- J15 pad 34: /DIO/DI3 -> /TempSens/Fan/TempAnalog
- J15 pad 35: /DIO/DO0 -> (no net)
- J15 pad 36: /DIO/DO1 -> /TempSens/Fan/TempAnalog_2
- J15 pad 38: (no net) -> /MCU/FPGA connection/PWM3n
- J15 pad 39: (no net) -> /MCU/FPGA connection/PWM0n
- J15 pad 40: (no net) -> /MCU/FPGA connection/PWM0p
- J15 pad 41: /CAN/RS485/RS485_TXEN -> /MCU/FPGA connection/PWM1n
- J15 pad 42: /CAN/RS485/RS485_TX -> /MCU/FPGA connection/PWM1p
- J15 pad 43: /CAN/RS485/RS485_RX -> /MCU/FPGA connection/PWM2n
- J15 pad 44: (no net) -> /MCU/FPGA connection/PWM2p
- J15 pad 45: /CAN/RS485/CAN_RX -> /MCU/FPGA connection/PWM3p
- J15 pad 46: /CAN/RS485/CAN_TX -> (no net)
- J15 pad 50: +3V3 -> /CAN/RS485/+5V
- J15 pad 9: /MCU/FPGA connection/Pulse -> (no net)
- J7 pad 2: /MOSFETs/CurSense/Isolation/Vpwr -> /Power DC/DC/+24VP
- J8 pad 1: /MOSFETs/CurSense/Isolation/HB0s -> GNDPWR
- J8 pad 2: /MOSFETs/CurSense/Isolation/HB1 -> /MOSFETs/CurSense/Isolation/Vpwr
- J9 pad 1: /CAN/RS485/CAN_H -> /MOSFETs/CurSense/Isolation/HB0s
- J9 pad 2: /CAN/RS485/CAN_L -> /MOSFETs/CurSense/Isolation/HB1
- J9 pad 3: GND -> /MOSFETs/CurSense/Isolation/HB2
- L1 pad 1: Net-(C24-Pad1) -> Net-(C22-Pad1)
- L1 pad 2: Net-(C30-Pad1) -> Net-(C28-Pad1)
- L2 pad 1: Net-(C30-Pad1) -> Net-(C28-Pad1)
- L3 pad 2: Net-(C33-Pad1) -> Net-(C31-Pad1)
- L4 pad 1: Net-(C33-Pad1) -> Net-(C31-Pad1)
- R46 pad 2: Net-(C33-Pad1) -> Net-(C31-Pad1)
- TP34 pad 1: Net-(C33-Pad1) -> Net-(C31-Pad1)
- U18 pad 1: Net-(C37-Pad1) -> Net-(C35-Pad1)
- U3 pad 1: /MOSFETs/CurSense/Isolation/HIN0 -> /DIO/+12V
- U3 pad 2: /MOSFETs/CurSense/Isolation/LIN0 -> /MOSFETs/CurSense/Isolation/HIN0
- U3 pad 3: GNDPWR -> /MOSFETs/CurSense/Isolation/LIN0
- U3 pad 4: Net-(R10-Pad2) -> GNDPWR
- U3 pad 5: /DIO/+12V -> Net-(R10-Pad2)
- U4 pad 1: /MOSFETs/CurSense/Isolation/HIN1 -> /DIO/+12V
- U4 pad 2: /MOSFETs/CurSense/Isolation/LIN1 -> /MOSFETs/CurSense/Isolation/HIN1
- U4 pad 3: GNDPWR -> /MOSFETs/CurSense/Isolation/LIN1
- U4 pad 4: Net-(R12-Pad2) -> GNDPWR
- U4 pad 5: /DIO/+12V -> Net-(R12-Pad2)
- U5 pad 1: /MOSFETs/CurSense/Isolation/HIN2 -> /DIO/+12V
- U5 pad 2: /MOSFETs/CurSense/Isolation/LIN2 -> /MOSFETs/CurSense/Isolation/HIN2
- U5 pad 3: GNDPWR -> /MOSFETs/CurSense/Isolation/LIN2
- U5 pad 4: Net-(R14-Pad2) -> GNDPWR
- U5 pad 5: /DIO/+12V -> Net-(R14-Pad2)
- U6 pad 1: /MOSFETs/CurSense/Isolation/HIN3 -> /DIO/+12V
- U6 pad 2: /MOSFETs/CurSense/Isolation/LIN3 -> /MOSFETs/CurSense/Isolation/HIN3
- U6 pad 3: GNDPWR -> /MOSFETs/CurSense/Isolation/LIN3
- U6 pad 4: Net-(R16-Pad2) -> GNDPWR
- U6 pad 5: /DIO/+12V -> Net-(R16-Pad2)
- U7 pad 1: /MOSFETs/CurSense/Isolation/HB0s -> /MOSFETs/CurSense/Isolation/HB0
- U7 pad 2: /MOSFETs/CurSense/Isolation/HB0s -> /MOSFETs/CurSense/Isolation/HB0
- U7 pad 3: /MOSFETs/CurSense/Isolation/HB0 -> /MOSFETs/CurSense/Isolation/HB0s
- U7 pad 4: /MOSFETs/CurSense/Isolation/HB0 -> /MOSFETs/CurSense/Isolation/HB0s
- U7 pad 6: Net-(C13-Pad1) -> GND
- U8 pad 1: /MOSFETs/CurSense/Isolation/HB2s -> /MOSFETs/CurSense/Isolation/HB3s
- U8 pad 2: /MOSFETs/CurSense/Isolation/HB2s -> /MOSFETs/CurSense/Isolation/HB3s
- U8 pad 3: /MOSFETs/CurSense/Isolation/HB2 -> /MOSFETs/CurSense/Isolation/HB3
- U8 pad 4: /MOSFETs/CurSense/Isolation/HB2 -> /MOSFETs/CurSense/Isolation/HB3
- U8 pad 6: Net-(C14-Pad1) -> GND
Routing:
- net /MOSFETs/CurSense/Isolation/Vpwr: track 102.4 -> 249.0 mm
- net GNDPWR: track 107.5 -> 1.46 mm
- net /MOSFETs/CurSense/Isolation/HB2: track 29.0 -> 95.9 mm
- net /MOSFETs/CurSense/Isolation/+5Vpwr: track 0.00 -> 63.2 mm
- net /MOSFETs/CurSense/Isolation/HB1: track 24.6 -> 75.2 mm
- net /DIO/+12V: track 80.2 -> 127.3 mm, vias 0 -> 5
- net /MOSFETs/CurSense/Isolation/HB0s: track 0.00 -> 44.0 mm
- net /MOSFETs/CurSense/Isolation/HB3s: track 0.00 -> 39.3 mm
- net Net-(C31-Pad1): track 0.00 -> 38.7 mm
- net Net-(D30-Pad1): track 0.00 -> 32.2 mm
- net (no net): track 0.00 -> 17.5 mm
- net Net-(D26-Pad1): track 0.00 -> 17.4 mm
- net Net-(C24-Pad1): track 17.1 -> 0.00 mm
- net Net-(C35-Pad1): track 0.00 -> 15.8 mm
- net /MOSFETs/CurSense/Isolation/HB3: track 28.9 -> 43.6 mm
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- removed copper zone on F.Cu, net /MOSFETs/CurSense/Isolation/HB0
- removed copper zone on F.Cu, net /MOSFETs/CurSense/Isolation/HB0s
- removed copper zone on F.Cu, net /MOSFETs/CurSense/Isolation/HB1
- removed copper zone on F.Cu, net /MOSFETs/CurSense/Isolation/HB2
- removed copper zone on F.Cu, net /MOSFETs/CurSense/Isolation/HB2s
- removed copper zone on F.Cu, net /MOSFETs/CurSense/Isolation/HB3
Other:
- board size 182 x 100 mm -> 150 x 100 mm

Commit message: upd
Parts:
- moved C36 141.1 mm to (90.4, 141.8), turned to 270 degrees
- moved C35 76.1 mm to (85.8, 140.0), turned to 270 degrees
- moved C40 25.2 mm to (134.2, 143.6)
- moved C38 19.6 mm to (110.2, 131.8), turned to 180 degrees
- moved C37 16.4 mm to (101.0, 132.0), turned to 90 degrees
- moved C41 6.15 mm to (121.6, 134.4)
- moved C39 5.84 mm to (107.6, 136.8)
- moved U19 5.79 mm to (108.6, 142.8)
- moved L5 5.21 mm to (98.8, 141.0)
- moved J7 5.00 mm to (54.2, 141.4)
- moved D28 3.91 mm to (71.6, 143.0)
- moved D29 2.92 mm to (80.6, 143.0)
Routing:
- net (no net): track 17.5 -> 0.00 mm
- net Net-(D30-Pad1): track 32.2 -> 20.3 mm
- net /Power DC/DC/+24VP: track 0.00 -> 11.2 mm
- net /MOSFETs/CurSense/Isolation/+5Vpwr: track 63.2 -> 73.8 mm
- net Net-(C35-Pad1): track 15.8 -> 24.1 mm
- net Net-(C31-Pad1): track 38.7 -> 42.4 mm
- net /DIO/+12V: track 127.3 -> 128.3 mm
- net /CAN/RS485/+5V: track 9.39 -> 8.50 mm

Commit message: upd
Parts:
- removed D31: NUP2105L, Package_TO_SOT_SMD:SOT-23
- removed J11: Spring_Terminal_Connector_01x03, TerminalBlock_KaiFeng:TerminalBlock_KaiFeng_KF141R-3_1x03_P2.54mm
- removed J13: Spring_Terminal_Connector_01x08, TerminalBlock_KaiFeng:TerminalBlock_KaiFeng_KF141R-8_1x08_P2.54mm
- removed JP1, JP2: Jumper_NC_Small, Connector_PinHeader_2.54mm:PinHeader_1x02_P2.54mm_Vertical
- removed Q9: 2N7002, Package_TO_SOT_SMD:SOT-23
- removed R19, R20, R21, R22: 33, Resistor_SMD:R_0603_1608Metric
- removed R53: 100, Resistor_SMD:R_0603_1608Metric
- removed R54, R55: 120, Resistor_SMD:R_0603_1608Metric
- removed TP21: SPI0_sck, TestPoint:TestPoint_Pad_D1.5mm
- removed TP22: SPI0_cs, TestPoint:TestPoint_Pad_D1.5mm
- removed TP23: SPI0_miso, TestPoint:TestPoint_Pad_D1.5mm
- removed TP24: SPI1_sck, TestPoint:TestPoint_Pad_D1.5mm
- removed TP25: SPI1_cs, TestPoint:TestPoint_Pad_D1.5mm
- removed TP26: SPI1_miso, TestPoint:TestPoint_Pad_D1.5mm
- removed TP38: CAN_Tx, TestPoint:TestPoint_Pad_D1.5mm
- removed TP39: CAN_Rx, TestPoint:TestPoint_Pad_D1.5mm
- removed TP40: 485_Tx, TestPoint:TestPoint_Pad_D1.5mm
- removed TP41: 485_Rx, TestPoint:TestPoint_Pad_D1.5mm
- removed TP42: 485_TxEn, TestPoint:TestPoint_Pad_D1.5mm
- removed U10, U9: ADS7886, Package_TO_SOT_SMD:SOT-23-6
- removed U20: SN65HVD230, Package_SOIC:SOIC-8_3.9x4.9mm_P1.27mm
- removed U21: MAX485CSA, Package_SOIC:SO-8_5.3x6.2mm_P1.27mm
- added C42: CP, Capacitor_THT:CP_Radial_D12.5mm_P5.00mm, F.Cu at (46.6, 173.9)
- added C43: CP, Capacitor_THT:CP_Radial_D12.5mm_P5.00mm, F.Cu at (61.1, 174.1)
- added C44: CP, Capacitor_SMD:C_2220_5650Metric_Pad2.02x5.50mm_HandSolder, B.Cu at (112.0, 133.0)
- added C45: CP, Capacitor_SMD:C_2220_5650Metric_Pad2.02x5.50mm_HandSolder, B.Cu at (112.1, 91.0)
- added C46: CP, Capacitor_SMD:C_2220_5650Metric_Pad2.02x5.50mm_HandSolder, B.Cu at (112.1, 105.0)
- added C47: CP, Capacitor_SMD:C_2220_5650Metric_Pad2.02x5.50mm_HandSolder, B.Cu at (112.0, 119.0)
- added C48: CP, Capacitor_THT:CP_Radial_D10.0mm_P5.00mm, B.Cu at (117.4, 88.2)
- added C49: CP, Capacitor_THT:CP_Radial_D10.0mm_P5.00mm, B.Cu at (117.4, 102.2)
- C1, C10, C11, C12, C13, C15, C17, C18, C19, C2, C20, C21, C22, C23, C24, C25, C26, C27, C28, C29, C3, C30, C31, C32, C33, C34, C35, C36, C37, C38, C39, C4, C5, C6, C7, C8, C9, D1, D10, D11, D12, D13, D14, D15, D16, D17, D18, D19, D2, D20, D21, D22, D23, D24, D25, D26, D27, D28, D29, D3, D30, D4, D5, D6, D7, D8, D9, F1, F2, F3, L1, L2, L3, L4, L5, MK1, MK2, MK3, MK4, Q10, Q11, Q12, R1, R10, R11, R12, R13, R14, R15, R16, R17, R18, R2, R23, R24, R25, R26, R27, R28, R29, R3, R30, R31, R32, R33, R34, R37, R38, R39, R4, R40, R41, R42, R43, R44, R45, R46, R47, R48, R49, R5, R50, R51, R52, R6, R7, R8, R9, TP1, TP10, TP11, TP12, TP13, TP14, TP15, TP16, TP17, TP18, TP19, TP2, TP20, TP27, TP28, TP29, TP3, TP30, TP31, TP32, TP33, TP34, TP35, TP36, TP37, TP4, TP5, TP6, TP7, TP8, TP9, U1, U11, U12, U13, U14, U15, U16, U17, U18, U19, U2, U3, U4, U5, U6, U7, U8: moved to B.Cu
- C14, C16: value 0.1uF -> CP; footprint Capacitor_SMD:C_0603_1608Metric -> Capacitor_THT:CP_Radial_D22.0mm_P10.00mm_SnapIn
- C40, C41: value 0.1uF -> CP; footprint Capacitor_SMD:C_0603_1608Metric -> Capacitor_THT:CP_Radial_D10.0mm_P5.00mm; moved to B.Cu
- J1, J2, J3, J4: value Spring_Terminal_Connector_01x03 -> Screw_Terminal_01x03; footprint TerminalBlock_KaiFeng:TerminalBlock_KaiFeng_KF141R-3_1x03_P2.54mm -> TerminalBlock:TerminalBlock_Altech_AK300-3_P5.00mm; moved to F.Cu
- J10: value Spring_Terminal_Connector_01x03 -> Conn_01x08; footprint TerminalBlock_KaiFeng:TerminalBlock_KaiFeng_KF141R-3_1x03_P2.54mm -> Connector_PinHeader_2.54mm:PinHeader_1x08_P2.54mm_Horizontal; moved to F.Cu
- J12: footprint TerminalBlock_KaiFeng:TerminalBlock_KaiFeng_KF141R-3_1x03_P2.54mm -> Connector_PinHeader_2.54mm:PinHeader_1x03_P2.54mm_Vertical; moved to F.Cu
- J14, J7, J8, J9, Q1, Q2, Q3, Q4, Q5, Q6, Q7, Q8, R35, R36: moved to F.Cu
- J15: value Conn_02x25_Odd_Even -> Conn_01x27; footprint Connector_PinHeader_2.54mm:PinHeader_2x25_P2.54mm_Vertical -> Connector_PinHeader_2.54mm:PinHeader_1x27_P2.54mm_Vertical; moved to F.Cu
- J16: value Conn_02x25_Odd_Even -> Conn_01x27; footprint Connector_PinHeader_2.54mm:PinHeader_2x25_P2.54mm_Vertical -> Connector_PinHeader_2.54mm:PinHeader_1x27_P2.54mm_Vertical
- J5, J6: value Spring_Terminal_Connector_01x02 -> Screw_Terminal_01x02; footprint TerminalBlock_KaiFeng:TerminalBlock_KaiFeng_KF141R-2_1x02_P2.54mm -> TerminalBlock:TerminalBlock_Altech_AK300-2_P5.00mm; moved to F.Cu
- moved TP27 289.3 mm to (64.0, 32.6), turned to 270 degrees
- moved C12 273.6 mm to (100.8, 146.7)
- moved C16 269.7 mm to (87.4, 136.8), turned to 180 degrees
- moved R39 257.3 mm to (163.5, 142.6)
- moved C21 244.4 mm to (182.6, 159.3)
- moved C10 233.0 mm to (105.3, 89.7)
- moved R38 229.6 mm to (162.9, 91.3)
- moved C14 228.6 mm to (87.4, 93.6), turned to 180 degrees
- moved R18 227.0 mm to (155.5, 149.4), turned to 180 degrees
- moved R42 226.7 mm to (169.4, 84.4), turned to 270 degrees
- moved R41 225.7 mm to (179.4, 85.7)
- moved C18 225.7 mm to (163.0, 145.3), turned to 270 degrees
- moved C3 222.7 mm to (142.0, 96.0), turned to 270 degrees
- moved R44 220.9 mm to (187.3, 92.5), turned to 180 degrees
- moved R43 219.6 mm to (183.4, 91.0), turned to 180 degrees
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Connections:
- C1 pad 2: +3V3 -> /Encoder Interface/+3.3V
- C10 pad 2: /CAN/RS485/+5V -> /Encoder Interface/+3.3V
- C12 pad 2: /CAN/RS485/+5V -> /Encoder Interface/+3.3V
- C14 pad 1: GND -> /MOSFETs/CurSense/Isolation/Vpwr
- C14 pad 2: /CAN/RS485/+5V -> GNDPWR
- C16 pad 1: GND -> /MOSFETs/CurSense/Isolation/Vpwr
- C16 pad 2: /CAN/RS485/+5V -> GNDPWR
- C2 pad 2: +3V3 -> /Encoder Interface/+3.3V
- C24 pad 1: /CAN/RS485/+5V -> /MCU/FPGA connection/+5V
- C26 pad 1: /CAN/RS485/+5V -> /MCU/FPGA connection/+5V
- C3 pad 1: GND -> GNDPWR
- C34 pad 1: +3V3 -> /Encoder Interface/+3.3V
- C4 pad 1: GND -> GNDPWR
- C40 pad 1: +3V3 -> /MOSFETs/CurSense/Isolation/Vpwr
- C40 pad 2: GND -> GNDPWR
- C41 pad 1: /CAN/RS485/+5V -> /MOSFETs/CurSense/Isolation/Vpwr
- C41 pad 2: GND -> GNDPWR
- J1 pad 1: /Power DC/DC/+24VP -> GNDPWR
- J1 pad 3: GNDPWR -> /Power DC/DC/+24VP
- J10 pad 1: /CAN/RS485/CAN_H -> /Encoder Interface/EncA-
- J10 pad 2: /CAN/RS485/CAN_L -> /Encoder Interface/EncA+
- J10 pad 3: GND -> /Encoder Interface/EncB-
- J15 pad 1: (no net) -> /MCU/FPGA connection/+5V
- J15 pad 10: GND -> /MCU/FPGA connection/PWM1p
- J15 pad 11: +3V3 -> /MCU/FPGA connection/PWM1n
- J15 pad 12: (no net) -> /Encoder Interface/+3.3V
- J15 pad 13: (no net) -> GND
- J15 pad 15: /MCU/FPGA connection/ADC_Csens0 -> /Encoder Interface/+3.3V
- J15 pad 16: (no net) -> GND
- J15 pad 17: /MCU/FPGA connection/ADC_Csens1 -> /MCU/FPGA connection/PWM2p
- J15 pad 18: (no net) -> /MCU/FPGA connection/PWM2n
- J15 pad 19: +3V3 -> GND
- J15 pad 2: (no net) -> /MCU/FPGA connection/ADC_Csens0
- J15 pad 20: (no net) -> /MCU/FPGA connection/PWM3p
- J15 pad 21: (no net) -> /MCU/FPGA connection/PWM3n
- J15 pad 22: +3V3 -> /Encoder Interface/+3.3V
- J15 pad 23: /Encoder Interface/EncA -> GND
- J15 pad 24: /Encoder Interface/EncB -> /TempSens/Fan/TempAnalog_2
- J15 pad 25: /Encoder Interface/EncZ -> GND
- J15 pad 26: (no net) -> /MCU/FPGA connection/ADC_Csens1
- J15 pad 27: GND -> /MCU/FPGA connection/+5V
- J15 pad 3: (no net) -> GND
- J15 pad 4: (no net) -> /TempSens/Fan/TempAnalog
- J15 pad 5: (no net) -> /Encoder Interface/+3.3V
- J15 pad 6: (no net) -> GND
- J15 pad 7: (no net) -> /MCU/FPGA connection/PWM0p
- J15 pad 8: (no net) -> /MCU/FPGA connection/PWM0n
- J15 pad 9: (no net) -> GND
- J16 pad 1: /MCU/FPGA connection/SPI1_CSn -> /MCU/FPGA connection/+5V
- J16 pad 10: (no net) -> /DIO/DI2
- J16 pad 11: (no net) -> /DIO/DI3
- J16 pad 12: (no net) -> /Encoder Interface/+3.3V
- J16 pad 13: /MCU/FPGA connection/PWM -> GND
- J16 pad 14: (no net) -> /MCU/FPGA connection/Vsense2
- J16 pad 15: (no net) -> /Encoder Interface/+3.3V
- J16 pad 16: (no net) -> GND
- J16 pad 17: (no net) -> /MCU/FPGA connection/PWM
- J16 pad 18: (no net) -> /MCU/FPGA connection/Pulse
- J16 pad 19: (no net) -> GND
- J16 pad 2: /MCU/FPGA connection/SPI1_SCK -> /DIO/DO0
- J16 pad 20: (no net) -> /Encoder Interface/EncZ
- J16 pad 21: (no net) -> /Encoder Interface/EncA
- J16 pad 22: (no net) -> /Encoder Interface/+3.3V
- J16 pad 23: +3V3 -> GND
- J16 pad 24: GND -> /Encoder Interface/EncB
- J16 pad 25: +3V3 -> GND
- J16 pad 27: (no net) -> /MCU/FPGA connection/+5V
- J16 pad 3: /MCU/FPGA connection/SPI1_MISO -> GND
- J16 pad 4: (no net) -> /DIO/DO1
- J16 pad 5: (no net) -> /Encoder Interface/+3.3V
- J16 pad 6: (no net) -> GND
- J16 pad 7: (no net) -> /DIO/DI0
- J16 pad 8: (no net) -> /DIO/DI1
- J16 pad 9: /MCU/FPGA connection/Pulse -> GND
- J2 pad 1: /Power DC/DC/+24VP -> GNDPWR
- J2 pad 3: GNDPWR -> /Power DC/DC/+24VP
- J3 pad 1: /Power DC/DC/+24VP -> GNDPWR
- J3 pad 3: GNDPWR -> /Power DC/DC/+24VP
- J4 pad 1: /Power DC/DC/+24VP -> GNDPWR
- J4 pad 3: GNDPWR -> /Power DC/DC/+24VP
- R1 pad 2: +3V3 -> /Encoder Interface/+3.3V
- R2 pad 2: +3V3 -> /Encoder Interface/+3.3V
- R3 pad 2: +3V3 -> /Encoder Interface/+3.3V
- R35 pad 2: +3V3 -> /Encoder Interface/+3.3V
- R36 pad 2: +3V3 -> /Encoder Interface/+3.3V
- R4 pad 2: +3V3 -> /Encoder Interface/+3.3V
- R44 pad 2: +3V3 -> /Encoder Interface/+3.3V
- R5 pad 2: +3V3 -> /Encoder Interface/+3.3V
- R6 pad 2: +3V3 -> /Encoder Interface/+3.3V
- R7 pad 2: +3V3 -> /Encoder Interface/+3.3V
- R8 pad 2: +3V3 -> /Encoder Interface/+3.3V
- TP31 pad 1: /CAN/RS485/+5V -> /MCU/FPGA connection/+5V
- U1 pad 1: +3V3 -> /Encoder Interface/+3.3V
- U1 pad 7: +3V3 -> /Encoder Interface/+3.3V
- U11 pad 5: Net-(D18-Pad2) -> Net-(D17-Pad2)
- U11 pad 7: Net-(D17-Pad2) -> Net-(D18-Pad2)
- U12 pad 1: Net-(R27-Pad1) -> Net-(R28-Pad1)
- U12 pad 3: Net-(R28-Pad1) -> Net-(R27-Pad1)
- U14 pad 2: /CAN/RS485/+5V -> /MCU/FPGA connection/+5V
- U17 pad 16: +3V3 -> /Encoder Interface/+3.3V
- U17 pad 4: +3V3 -> /Encoder Interface/+3.3V
- U2 pad 1: +3V3 -> /Encoder Interface/+3.3V
- U2 pad 7: +3V3 -> /Encoder Interface/+3.3V
- U7 pad 8: /CAN/RS485/+5V -> /Encoder Interface/+3.3V
- U8 pad 8: /CAN/RS485/+5V -> /Encoder Interface/+3.3V
Routing:
- net /MOSFETs/CurSense/Isolation/Vpwr: track 249.0 -> 68.0 mm
- net /Encoder Interface/+3.3V: track 0.00 -> 159.7 mm, vias 0 -> 3
- net /MOSFETs/CurSense/Isolation/HB2: track 95.9 -> 21.0 mm
- net Net-(R17-Pad2): track 0.00 -> 63.2 mm, vias 0 -> 2
- net GND: track 0.00 -> 62.0 mm
- net /MCU/FPGA connection/PWM: track 0.00 -> 56.4 mm
- net Net-(R18-Pad2): track 0.00 -> 55.4 mm
- net /MOSFETs/CurSense/Isolation/HB1: track 75.2 -> 20.4 mm
- net Net-(R26-Pad1): track 0.00 -> 54.0 mm, vias 0 -> 2
- net Net-(R25-Pad1): track 0.00 -> 52.5 mm, vias 0 -> 2
- net /DIO/DI3: track 0.00 -> 46.8 mm
- net /MCU/FPGA connection/Pulse: track 0.00 -> 44.3 mm
- net /MOSFETs/CurSense/Isolation/HB0s: track 44.0 -> 0.00 mm
- net /DIO/DI2: track 0.00 -> 41.6 mm
- net /DIO/DI1: track 0.00 -> 40.1 mm, vias 0 -> 1
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- added copper zone on B.Cu, net /MOSFETs/CurSense/Isolation/HB0
- added copper zone on B.Cu, net /MOSFETs/CurSense/Isolation/HB0s
- added copper zone on B.Cu, net /MOSFETs/CurSense/Isolation/HB1
- added copper zone on B.Cu, net /MOSFETs/CurSense/Isolation/HB2
- added copper zone on B.Cu, net /MOSFETs/CurSense/Isolation/HB3
- added copper zone on B.Cu, net /MOSFETs/CurSense/Isolation/HB3s
- added copper zone on F.Cu, net /MOSFETs/CurSense/Isolation/Vpwr
- added copper zone on F.Cu, net GNDPWR
Other:
- net class Default: clearance 0.4 -> 0.45
- rule trace_clearance: 0.4 -> 0.45

Commit message: upd
Parts:
- added R19: 10k, Resistor_SMD:R_0603_1608Metric, B.Cu at (208.7, 135.6)
- added R20: 10k, Resistor_SMD:R_0603_1608Metric, B.Cu at (208.7, 143.2)
- added R21: 10k, Resistor_SMD:R_0603_1608Metric, B.Cu at (208.7, 133.0)
- moved R44 41.1 mm to (208.7, 127.6), turned to 0 degrees
- moved D22 40.7 mm to (209.6, 129.5), turned to 0 degrees
- moved R42 13.0 mm to (181.0, 90.2)
- moved Q12 12.3 mm to (184.0, 90.2)
- moved R41 8.44 mm to (183.8, 92.9)
- moved R43 6.01 mm to (187.8, 95.1)
- moved U12 3.30 mm to (186.1, 78.6)
- moved U15 3.30 mm to (178.0, 157.0)
- moved C27 2.94 mm to (184.6, 156.9)
- moved C21 2.91 mm to (185.5, 159.6)
- moved C20 2.30 mm to (178.7, 95.1)
- moved C26 2.20 mm to (177.9, 92.8)
- moved J12 0.50 mm to (155.1, 88.2)
Connections:
- J14 pad 1: GND -> /Digital DC/DC/+24VD
- J14 pad 2: /Digital DC/DC/+24VD -> GND
Routing:
- net /Power DC/DC/+24VP: track 0.00 -> 142.7 mm
- net /Encoder Interface/+3.3V: track 159.7 -> 298.7 mm, vias 3 -> 4
- net /Digital DC/DC/+6.8V: track 7.56 -> 80.1 mm, vias 0 -> 2
- net /Digital DC/DC/+Vpp: track 5.70 -> 70.4 mm, vias 0 -> 2
- net /Encoder Interface/EncZ: track 0.00 -> 19.7 mm, vias 0 -> 1
- net /TempSens/Fan/FAN_PWR: track 20.0 -> 36.9 mm
- net /Digital DC/DC/+5VEnc: track 0.00 -> 13.6 mm
- net /Encoder Interface/EncB: track 0.08 -> 12.2 mm
- net /Encoder Interface/EncA: track 0.02 -> 11.6 mm
- net /MCU/FPGA connection/PWM: track 56.4 -> 46.1 mm
- net /DIO/DI1: track 40.1 -> 30.2 mm, vias 1 -> 0
- net /MCU/FPGA connection/Vsense2: track 0.14 -> 8.87 mm
- net /DIO/DI0: track 38.3 -> 31.0 mm
- net /TempSens/Fan/FAN_PULSE: track 39.5 -> 46.2 mm
- net Net-(Q12-Pad1): track 9.29 -> 3.78 mm
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- added copper zone on F.Cu, net GND
Other:
- board text added: "Hall mode"

Commit message: upd
Parts:
- moved R35 0.20 mm to (141.5, 112.0)
Routing:
- net /Power DC/DC/+24VP: track 142.7 -> 144.4 mm

Commit message: upd
Parts:
- removed TP10: PWM1p, TestPoint:TestPoint_Pad_D1.5mm
- removed TP11: PWM1n, TestPoint:TestPoint_Pad_D1.5mm
- removed TP12: PWM2p, TestPoint:TestPoint_Pad_D1.5mm
- removed TP13: PWM2n, TestPoint:TestPoint_Pad_D1.5mm
- removed TP14: PWM3p, TestPoint:TestPoint_Pad_D1.5mm
- removed TP15: PWM3n, TestPoint:TestPoint_Pad_D1.5mm
- removed TP2: GNDp, TestPoint:TestPoint_Pad_D1.5mm
- removed TP27: driver_VB, TestPoint:TestPoint_Pad_D1.5mm
- removed TP28: driver_VS, TestPoint:TestPoint_Pad_D1.5mm
- removed TP29: driver_HO, TestPoint:TestPoint_Pad_D1.5mm
- removed TP31: +5Vd_main, TestPoint:TestPoint_Pad_D1.5mm
- removed TP33: +24Vd_OUT, TestPoint:TestPoint_Pad_D1.5mm
- removed TP34: +6.8Vd, TestPoint:TestPoint_Pad_D1.5mm
- removed TP35: +24Vp_IN, TestPoint:TestPoint_Pad_D1.5mm
- removed TP36: +12Vp, TestPoint:TestPoint_Pad_D1.5mm
- removed TP37: +5Vp, TestPoint:TestPoint_Pad_D1.5mm
- removed TP6: Csen_0, TestPoint:TestPoint_Pad_D1.5mm
- removed TP7: Csen_1, TestPoint:TestPoint_Pad_D1.5mm
- removed TP8: PWM0p, TestPoint:TestPoint_Pad_D1.5mm
- removed TP9: PWM0n, TestPoint:TestPoint_Pad_D1.5mm
- TP16, TP17, TP18, TP19, TP20, TP4, TP5: moved to F.Cu
- moved TP18 147.5 mm to (200.4, 157.6)
- moved TP17 145.7 mm to (203.6, 157.4)
- moved TP32 129.8 mm to (177.8, 156.2)
- moved TP16 128.8 mm to (215.7, 123.5)
- moved TP3 118.3 mm to (136.7, 154.7)
- moved TP4 114.2 mm to (136.7, 154.6)
- moved TP19 90.0 mm to (150.2, 118.0)
- moved TP20 82.6 mm to (150.2, 117.9)
- moved TP30 81.0 mm to (157.6, 154.7)
- moved TP5 64.4 mm to (138.8, 99.5)
- moved C42 57.9 mm to (100.4, 152.4)
- moved C43 53.0 mm to (109.5, 152.6)
- moved TP1 47.2 mm to (75.7, 70.7)
- moved C48 0.30 mm to (117.4, 87.9)
- moved C49 0.28 mm to (117.2, 102.0)
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Routing:
- net GND: track 62.0 -> 181.0 mm, vias 0 -> 5
- net GNDPWR: track 8.64 -> 68.1 mm, vias 3 -> 5
- net /DIO/+12V: track 147.2 -> 169.9 mm
- net /Encoder Interface/+3.3V: track 298.4 -> 317.7 mm
- net Net-(C31-Pad1): track 26.9 -> 41.1 mm
- net Net-(C28-Pad1): track 15.6 -> 27.4 mm
- net /MOSFETs/CurSense/Isolation/Vpwr: track 68.0 -> 78.9 mm
- net /MOSFETs/CurSense/Isolation/HB0: track 20.8 -> 29.1 mm
- net Net-(R45-Pad1): track 0.00 -> 6.60 mm
- net /MOSFETs/CurSense/Isolation/HB2: track 21.0 -> 24.9 mm
- net /MOSFETs/CurSense/Isolation/HB1: track 20.4 -> 24.3 mm
- net /MOSFETs/CurSense/Isolation/HB3: track 20.9 -> 24.6 mm
- net /Digital DC/DC/+5VEnc: track 13.6 -> 16.6 mm
- net /Encoder Interface/EncB-: track 14.4 -> 17.2 mm
- net /Encoder Interface/EncZ+: track 21.7 -> 24.5 mm
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- added copper zone on B.Cu, net GND
- added copper zone on B.Cu, net GNDPWR

Commit message: current version
Parts:
- removed TP20: GNDd, TestPoint:TestPoint_Pad_D1.5mm
- removed TP30: +24Vd_IN, TestPoint:TestPoint_Pad_D1.5mm
- removed TP5: GNDp, TestPoint:TestPoint_Pad_D1.5mm
- added TP2: GNDp, TestPoint:TestPoint_Pad_D1.5mm, F.Cu at (76.8, 115.8)
- added TP31: +5Vd_main, TestPoint:TestPoint_Pad_D1.5mm, B.Cu at (163.0, 85.1)
- added TP33: +24Vd_OUT, TestPoint:TestPoint_Pad_D1.5mm, B.Cu at (197.9, 115.8)
- added TP34: +6.8Vd, TestPoint:TestPoint_Pad_D1.5mm, B.Cu at (188.1, 119.9)
- added TP36: +12Vp, TestPoint:TestPoint_Pad_D1.5mm, B.Cu at (123.2, 80.2)
- added TP37: +5Vp, TestPoint:TestPoint_Pad_D1.5mm, B.Cu at (137.1, 84.1)
- D13, D14, D15, D16: footprint LED_SMD:LED_0603_1608Metric -> LED_SMD:LED_0603_1608Metric_ReverseMount
- moved TP32 5.13 mm to (177.7, 151.1)
- moved C42 2.78 mm to (99.0, 154.8), turned to 180 degrees
- moved TP17 1.15 mm to (204.7, 157.7)
Routing:
- net Net-(C31-Pad1): track 41.1 -> 49.8 mm
- net /MOSFETs/CurSense/Isolation/+5Vpwr: track 76.3 -> 81.6 mm
- net /MCU/FPGA connection/+5V: track 22.4 -> 25.7 mm
- net /DIO/+12V: track 169.9 -> 172.9 mm
- net GNDPWR: track 68.1 -> 71.0 mm
- net /Digital DC/DC/+Vpp: track 70.4 -> 72.9 mm
- net Net-(R26-Pad1): track 54.7 -> 56.9 mm
- net GND: track 181.0 -> 183.0 mm, vias 5 -> 6
- net Net-(C5-Pad1): track 5.13 -> 6.07 mm
