File: base/dio.sch (KiCad schematic (older format))
At the start: 26 parts, among them Q10 2N7002, Q11 2N7002, Q9 2N7002, U11 MOCD217M, U12 MOCD217M, U13 MOCD217M

Commit message: upd
Parts:
- removed Q9: 2N7002, Package_TO_SOT_SMD:SOT-23, symbol Q_NMOS_GSD
Connections:
- wire segments 65 -> 70
Other:
- moved on the sheet: D13, D14, R27, R28
Changed lines of the file:
@@
 $Descr A4 11693 8268
 encoding utf-8
-Sheet 3 9
+Sheet 3 8
 Title ""
 Date ""
@@
 Comment4 ""
 $EndDescr
-Text HLabel 2850 4900 0    60   Input ~ 0
+Text HLabel 2850 5350 0    60   Input ~ 0
 DI0_P
-Text HLabel 2850 5350 0    60   Input ~ 0
+Text HLabel 2900 4900 0    60   Input ~ 0
 DI1_P
 Text HLabel 2850 5850 0    60   Input ~ 0
@@
 L LED D13
 U 1 1 5A43CD4D
-P 3100 4900
-F 0 "D13" H 3100 5000 50  0000 C CNN
-F 1 "LED" H 3100 4800 50  0000 C CNN
-F 2 "LED_SMD:LED_0603_1608Metric" H 3100 4900 50  0001 C CNN
-F 3 "" H 3100 4900 50  0001 C CNN
-	1    3100 4900
-	-1   0    0    1
-$EndComp
-$Comp
-L R R27
-U 1 1 5A43CDFC
-P 3500 4900
-F 0 "R27" V 3580 4900 50  0000 C CNN
-F 1 "2k2" V 3500 4900 50  0000 C CNN
-F 2 "Resistor_SMD:R_0603_1608Metric" V 3430 4900 50  0001 C CNN
-F 3 "" H 3500 4900 50  0001 C CNN
-	1    3500 4900
-	0    1    1    0
-$EndComp
-$Comp
-L LED D14
-U 1 1 5A43CE85
 P 3100 5350
-F 0 "D14" H 3100 5450 50  0000 C CNN
+F 0 "D13" H 3100 5450 50  0000 C CNN
 F 1 "LED" H 3100 5250 50  0000 C CNN
 F 2 "LED_SMD:LED_0603_1608Metric" H 3100 5350 50  0001 C CNN
@@
 $EndComp
 $Comp
-L R R28
-U 1 1 5A43CEB2
+L R R27
+U 1 1 5A43CDFC
 P 3500 5350
-F 0 "R28" V 3580 5350 50  0000 C CNN
+F 0 "R27" V 3580 5350 50  0000 C CNN
 F 1 "2k2" V 3500 5350 50  0000 C CNN
 F 2 "Resistor_SMD:R_0603_1608Metric" V 3430 5350 50  0001 C CNN
 F 3 "" H 3500 5350 50  0001 C CNN
 	1    3500 5350
+	0    1    1    0
+$EndComp
+$Comp
+L LED D14
+U 1 1 5A43CE85
+P 3150 4900
+F 0 "D14" H 3150 5000 50  0000 C CNN
+F 1 "LED" H 3150 4800 50  0000 C CNN
+F 2 "LED_SMD:LED_0603_1608Metric" H 3150 4900 50  0001 C CNN
+F 3 "" H 3150 4900 50  0001 C CNN
+	1    3150 4900
+	-1   0    0    1
+$EndComp
+$Comp
+L R R28
+U 1 1 5A43CEB2
+P 3550 4900
+F 0 "R28" V 3630 4900 50  0000 C CNN
+F 1 "2k2" V 3550 4900 50  0000 C CNN
+F 2 "Resistor_SMD:R_0603_1608Metric" V 3480 4900 50  0001 C CNN
+F 3 "" H 3550 4900 50  0001 C CNN
+	1    3550 4900
 	0    1    1    0
 $EndComp
@@
 GNDP
 Wire Wire Line
-	2850 4900 2950 4900
-Wire Wire Line
-	3250 4900 3350 4900
-Wire Wire Line
-	3650 4900 3850 4900
-Wire Wire Line
 	2850 5350 2950 5350
 Wire Wire Line
 	3250 5350 3350 5350
 Wire Wire Line
-	3650 5350 3850 5350
+	2900 4900 3000 4900
+Wire Wire Line
+	3300 4900 3400 4900
 Wire Wire Line
 	2850 5850 2950 5850
@@
 	1050 1050 1750 1050
 Wire Wire Line
-	3950 2000 4950 2000
-Wire Wire Line
 	4350 2050 4350 2000
 Connection ~ 4350 2000
@@
 	6200 1650 6550 1650
 Wire Wire Line
-	3950 3350 4950 3350
-Wire Wire Line
-	4350 3400 4350 3350
+	4350 2900 4350 3400
 Connection ~ 4350 3350
 Wire Wire Line
@@
 Text Label 2300 3350 0    60   ~ 0
 GNDD
-$Comp
-L Q_NMOS_GSD Q9
-U 1 1 5A455FDA
-P 3750 1900
-F 0 "Q9" H 3950 1950 50  0000 L CNN
-F 1 "2N7002" H 3950 1850 50  0000 L CNN
-F 2 "Package_TO_SOT_SMD:SOT-23" H 3950 2000 50  0001 C CNN
-F 3 "" H 3750 1900 50  0001 C CNN
-	1    3750 1900
-	1    0    0    -1
-$EndComp
+Wire Wire Line
+	3950 3350 4250 3350
+Wire Wire Line
+	4250 3350 4250 2000
+Wire Wire Line
+	4250 2000 4950 2000
+Wire Wire Line
+	3950 2000 4050 2000
+Wire Wire Line
+	4050 2000 4050 2900
+Wire Wire Line
+	4050 2900 4350 2900
+Wire Wire Line
+	4350 3350 4950 3350
+Wire Wire Line
+	3850 5350 3650 5350
+Wire Wire Line
+	3850 4900 3700 4900
 $EndSCHEMATC

Commit message: current version
Parts:
- D13, D14, D15, D16: footprint LED_SMD:LED_0603_1608Metric -> LED_SMD:LED_0603_1608Metric_ReverseMount
Changed lines of the file:
@@
 F 0 "D13" H 3100 5450 50  0000 C CNN
 F 1 "LED" H 3100 5250 50  0000 C CNN
-F 2 "LED_SMD:LED_0603_1608Metric" H 3100 5350 50  0001 C CNN
+F 2 "LED_SMD:LED_0603_1608Metric_ReverseMount" H 3100 5350 50  0001 C CNN
 F 3 "" H 3100 5350 50  0001 C CNN
 	1    3100 5350
@@
 F 0 "D14" H 3150 5000 50  0000 C CNN
 F 1 "LED" H 3150 4800 50  0000 C CNN
-F 2 "LED_SMD:LED_0603_1608Metric" H 3150 4900 50  0001 C CNN
+F 2 "LED_SMD:LED_0603_1608Metric_ReverseMount" H 3150 4900 50  0001 C CNN
 F 3 "" H 3150 4900 50  0001 C CNN
 	1    3150 4900
@@
 F 0 "D15" H 3100 5950 50  0000 C CNN
 F 1 "LED" H 3100 5750 50  0000 C CNN
-F 2 "LED_SMD:LED_0603_1608Metric" H 3100 5850 50  0001 C CNN
+F 2 "LED_SMD:LED_0603_1608Metric_ReverseMount" H 3100 5850 50  0001 C CNN
 F 3 "" H 3100 5850 50  0001 C CNN
 	1    3100 5850
@@
 F 0 "D16" H 3100 6400 50  0000 C CNN
 F 1 "LED" H 3100 6200 50  0000 C CNN
-F 2 "LED_SMD:LED_0603_1608Metric" H 3100 6300 50  0001 C CNN
+F 2 "LED_SMD:LED_0603_1608Metric_ReverseMount" H 3100 6300 50  0001 C CNN
 F 3 "" H 3100 6300 50  0001 C CNN
 	1    3100 6300

Commit message: add power vias
Parts:
- D17, D18: footprint LED_SMD:LED_0603_1608Metric -> LED_SMD:LED_0603_1608Metric_ReverseMount
Changed lines of the file:
@@
 F 0 "D17" H 4350 2300 50  0000 C CNN
 F 1 "LED" H 4350 2100 50  0000 C CNN
-F 2 "LED_SMD:LED_0603_1608Metric" H 4350 2200 50  0001 C CNN
+F 2 "LED_SMD:LED_0603_1608Metric_ReverseMount" H 4350 2200 50  0001 C CNN
 F 3 "" H 4350 2200 50  0001 C CNN
 	1    4350 2200
@@
 F 0 "D18" H 4350 3650 50  0000 C CNN
 F 1 "LED" H 4350 3450 50  0000 C CNN
-F 2 "LED_SMD:LED_0603_1608Metric" H 4350 3550 50  0001 C CNN
+F 2 "LED_SMD:LED_0603_1608Metric_ReverseMount" H 4350 3550 50  0001 C CNN
 F 3 "" H 4350 3550 50  0001 C CNN
 	1    4350 3550
