File: core_sf/core_sf.sch (KiCad schematic (older format))
At the start: 114 parts, among them J1 Conn_01x27, J2 Conn_01x27, J3 HR911105A, J4 HR911105A, J5 Conn_02x05_Odd_Even, J6 Screw_Terminal_01x03, J7 Screw_Terminal_01x03, U1 10M02SCE144, U2 LAN8720A, U3 LAN8720A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

Commit message: update core pinout
Connections:
- wire segments 512 -> 726

Commit message: debug design
Parts:
- added J10: Conn_01x04, Connector_PinHeader_2.54mm:PinHeader_1x04_P2.54mm_Vertical, symbol Conn_01x04
- added J8, J9: Conn_01x20, Connector_PinHeader_2.54mm:PinHeader_1x20_P2.54mm_Vertical, symbol Conn_01x20
Connections:
- net labels added: canRX, canTx, uartRx, uartTx
- wire segments 726 -> 556
Other:
- moved on the sheet: J1, J2
