File: core_sf/core_sf.kicad_pcb (KiCad board)
At the start: 2 copper layers, 114 parts, among them J1 Conn_01x27, J2 Conn_01x27, J3 HR911105A, J4 HR911105A, J5 Conn_02x05_Odd_Even, J6 Screw_Terminal_01x03, J7 Screw_Terminal_01x03, U1 10M02SCE144, U2 LAN8720A, U3 LAN8720A, U4 AMS1117-3.3, U5 AMS1117-3.3, U6 STM32F427VGTx, U7 SN65HVD230, U8 MAX485E, X1 DSC6011CI2A-008.0000

Commit message: debug design
Parts:
- removed C1, C31, C9: 470pF, Capacitor_SMD:C_0603_1608Metric
- removed C10, C11, C13, C15, C16, C17, C18, C19, C2, C20, C21, C22, C23, C24, C25, C26, C27, C28, C29, C3, C30, C32, C33, C34, C35, C36, C37, C38, C39, C40, C41, C42, C43, C44, C45, C46, C47, C48, C49, C5, C53, C54, C55, C56, C58, C59, C6, C61, C62, C63, C64, C65, C66, C8: 0.1uF, Capacitor_SMD:C_0603_1608Metric
- removed C12, C57: 220uF 4V, Capacitor_Tantalum_SMD:CP_EIA-3528-21_Kemet-B
- removed C14, C4, C51, C52, C60: 4.7uF 6.3V, Capacitor_SMD:C_0603_1608Metric
- removed C50, C7: 22uF 6.3V, Capacitor_Tantalum_SMD:CP_EIA-3216-18_Kemet-A
- removed J3, J4: HR911105A, Connector_RJ:RJ45_HR911105A
- removed J5: Conn_02x05_Odd_Even, Connector_PinHeader_1.27mm:PinHeader_2x05_P1.27mm_Vertical_SMD
- removed J6, J7: Screw_Terminal_01x03, TerminalBlock:TerminalBlock_Altech_AK300-3_P5.00mm
- removed JP1, JP2: Jumper, Connector_PinHeader_2.54mm:PinHeader_1x02_P2.54mm_Vertical
- removed L1, L2, L3, L4, L5: BLM18PG331SN1D, Inductor_SMD:L_0603_1608Metric
- removed R1, R10, R13, R14, R15, R4, R5, R6: 49R9, Resistor_SMD:R_0603_1608Metric
- removed R11, R19, R22, R23, R24, R25, R3, R9: 10K, Resistor_SMD:R_0603_1608Metric
- removed R12, R2: 12K1, Resistor_SMD:R_0603_1608Metric
- removed R16, R17, R7, R8: 680R, Resistor_SMD:R_0603_1608Metric
- removed R18: 100, Resistor_SMD:R_0603_1608Metric
- removed R20, R21: 120, Resistor_SMD:R_0603_1608Metric
- removed U1: 10M02SCE144, Package_QFP:LQFP-144-1EP_20x20mm_P0.5mm_EP4x4mm
- removed U2, U3: LAN8720A, Package_DFN_QFN:QFN-24-1EP_4x4mm_P0.5mm
- removed U4, U5: AMS1117-3.3, Package_TO_SOT_SMD:SOT-223-3_TabPin2
- removed U6: STM32F427VGTx, Package_QFP:LQFP-100_14x14mm_P0.5mm
- removed U7: SN65HVD230, Package_SOIC:SOIC-8_3.9x4.9mm_P1.27mm
- removed U8: MAX485E, Package_SOIC:SOIC-8_3.9x4.9mm_P1.27mm
- removed X1: DSC6011CI2A-008.0000, Oscillator:Oscillator_SMD_EuroQuartz_XO32-4pin_3.2x2.5mm
- added J10: Conn_01x04, Connector_PinHeader_2.54mm:PinHeader_1x04_P2.54mm_Vertical, F.Cu at (82.5, 132.1)
- added J8: Conn_01x20, Connector_PinHeader_2.54mm:PinHeader_1x20_P2.54mm_Vertical, F.Cu at (96.5, 129.5)
- added J9: Conn_01x20, Connector_PinHeader_2.54mm:PinHeader_1x20_P2.54mm_Vertical, F.Cu at (111.8, 129.5)
Connections:
- J1 pad 10: (no net) -> /TIM1_CH3
- J1 pad 11: (no net) -> /TIM1_CH3N
- J1 pad 12: (no net) -> +3V3
- J1 pad 13: (no net) -> GND
- J1 pad 14: (no net) -> /TIM1_BKIN
- J1 pad 15: (no net) -> +3V3
- J1 pad 16: (no net) -> GND
- J1 pad 17: (no net) -> /TIM1_CH2
- J1 pad 18: (no net) -> /TIM1_CH2N
- J1 pad 19: (no net) -> GND
- J1 pad 2: (no net) -> /ADC3_IN10
- J1 pad 20: (no net) -> /TIM1_CH1
- J1 pad 21: (no net) -> /TIM1_CH1N
- J1 pad 22: (no net) -> +3V3
- J1 pad 23: (no net) -> GND
- J1 pad 24: (no net) -> /ADC1_IN4
- J1 pad 25: (no net) -> GND
- J1 pad 26: (no net) -> /ADC2_IN9
- J1 pad 3: (no net) -> GND
- J1 pad 4: (no net) -> /ADC1_IN0
- J1 pad 5: (no net) -> +3V3
- J1 pad 6: (no net) -> GND
- J1 pad 7: (no net) -> /TIM1_CH4
- J1 pad 8: (no net) -> /TIM1_CH4N
- J1 pad 9: (no net) -> GND
- J2 pad 10: (no net) -> /GPIO4
- J2 pad 11: (no net) -> /GPIO5
- J2 pad 12: (no net) -> +3V3
- J2 pad 13: (no net) -> GND
- J2 pad 14: (no net) -> /ADC1_IN3
- J2 pad 15: (no net) -> +3V3
- J2 pad 16: (no net) -> GND
- J2 pad 17: (no net) -> /TIM3_FAN_PWM
- J2 pad 18: (no net) -> /TIM2_FAN_PULSE
- J2 pad 19: (no net) -> GND
- J2 pad 2: (no net) -> /GPIO0
- J2 pad 20: (no net) -> /TIM4_ENC_Z
- J2 pad 21: (no net) -> /TIM4_ENC_A
- J2 pad 22: (no net) -> +3V3
- J2 pad 23: (no net) -> GND
- J2 pad 24: (no net) -> /TIM4_ENC_B
- J2 pad 25: (no net) -> GND
- J2 pad 26: (no net) -> /GPIO6
- J2 pad 3: (no net) -> GND
- J2 pad 4: (no net) -> /GPIO1
- J2 pad 5: (no net) -> +3V3
- J2 pad 6: (no net) -> GND
- J2 pad 7: (no net) -> /GPIO2
- J2 pad 8: (no net) -> /GPIO3
- J2 pad 9: (no net) -> GND
Routing:
- net +5V: track 0.00 -> 207.4 mm, vias 0 -> 3
- net +3V3: track 0.00 -> 175.8 mm, vias 0 -> 4
- net /TIM1_CH1N: track 0.00 -> 68.6 mm, vias 0 -> 1
- net /ADC1_IN0: track 0.00 -> 66.2 mm, vias 0 -> 1
- net /ADC3_IN10: track 0.00 -> 64.3 mm, vias 0 -> 1
- net GND: track 0.00 -> 55.9 mm, vias 0 -> 12
- net /ADC1_IN4: track 0.00 -> 53.6 mm, vias 0 -> 1
- net /TIM1_CH2N: track 0.00 -> 48.5 mm, vias 0 -> 1
- net /ADC2_IN9: track 0.00 -> 48.5 mm, vias 0 -> 1
- net /TIM1_CH1: track 0.00 -> 47.2 mm, vias 0 -> 1
- net /TIM4_ENC_Z: track 0.00 -> 45.9 mm, vias 0 -> 1
- net /TIM4_ENC_A: track 0.00 -> 42.0 mm, vias 0 -> 1
- net /TIM1_CH2: track 0.00 -> 39.5 mm, vias 0 -> 1
- net /canRX: track 0.00 -> 38.9 mm
- net /TIM4_ENC_B: track 0.00 -> 36.1 mm, vias 0 -> 1
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- added copper zone on B.Cu, net GND
- added copper zone on F.Cu, net GND
Other:
- net class Default: clearance 0.2 -> 0.45; trace_width 0.25 -> 0.8; via_dia 0.6 -> 2.2
- rule trace_clearance: 0.2 -> 0.45
- rule trace_min: 0.2 -> 0.7
- rule via_min_drill: 0.3 -> 0.4
- rule via_min_size: 0.4 -> 1.2
- board text added: "svtmishin"

Commit message: debug core was prepared to rezonit
Parts:
- added C1: 470pF, Capacitor_SMD:C_0603_1608Metric, F.Cu at (80.8, 76.1)
- added C12: 220uF 4V, Capacitor_Tantalum_SMD:CP_EIA-3528-21_Kemet-B, F.Cu at (83.2, 106.0)
- added C2: 0.1uF, Capacitor_SMD:C_0603_1608Metric, F.Cu at (87.7, 110.9)
- added C5: 0.1uF, Capacitor_SMD:C_0603_1608Metric, F.Cu at (88.1, 76.2)
- added C7: 22uF 6.3V, Capacitor_Tantalum_SMD:CP_EIA-3216-18_Kemet-A, F.Cu at (84.0, 128.7)
- added C7: 22uF 6.3V, Capacitor_Tantalum_SMD:CP_EIA-3216-18_Kemet-A, F.Cu at (84.5, 76.9)
Routing:
- net +3V3: track 175.8 -> 219.0 mm, vias 4 -> 1
- net GND: track 55.9 -> 17.3 mm, vias 12 -> 5
- net /TIM1_CH1N: track 68.6 -> 53.5 mm, vias 1 -> 0
- net +5V: track 207.4 -> 216.3 mm, vias 3 -> 2
- net /TIM4_ENC_A: track 42.0 -> 45.8 mm
- net /TIM1_CH2N: track 48.5 -> 46.0 mm
- net /ADC1_IN0: track 66.2 -> 68.4 mm, vias 1 -> 0
- net /ADC3_IN10: track 64.3 -> 62.6 mm, vias 1 -> 0
- net /TIM1_CH1: track 47.2 -> 48.9 mm
- net /TIM4_ENC_B: track 36.1 -> 37.5 mm, vias 1 -> 0
- net /TIM3_FAN_PWM: track 19.2 -> 18.0 mm, vias 1 -> 0
- net /ADC2_IN9: track 48.5 -> 47.6 mm, vias 1 -> 0
- net /ADC1_IN4: track 53.6 -> 52.9 mm, vias 1 -> 0
- net /TIM1_CH2: track 39.5 -> 40.1 mm
- net /TIM4_ENC_Z: track 45.9 -> 45.7 mm, vias 1 -> 0
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Other:
- net class Default: via_dia 2.2 -> 0.8
- rule trace_min: 0.7 -> 0.4
- rule via_min_size: 1.2 -> 0.8

Commit message: migration to kicad 6
Other:
- net class Default removed
